File: MM27/MM27.kicad_pcb (KiCad board)
At the start: 2 copper layers, 14 parts, among them J1 B2B-PH-K-S, J2 B2B-PH-K-S, J3 Conn_01x06_Pin, J4 Conn_01x06_Pin, SW1 CL-SB-12A-01T, U1 AZ1117IH-3.3TRG1, U5 L293DD

Commit message: ir circuits
Parts:
- added C20: CL21B104KBCNNNC, Capacitor_SMD:C_0805_2012Metric, F.Cu at (151.3, 46.0)
- added C21: CL21A475KAQNNNE, Capacitor_SMD:C_0805_2012Metric, F.Cu at (151.3, 49.0)
- added LED5: INL-5AMIR15, LED_THT:LED_D3.0mm, F.Cu at (144.9, 47.2)
- added Q1: SFH 313 FA-3/4, LED_THT:LED_D3.0mm, F.Cu at (144.9, 52.7)
- added Q10: NMOS, Package_TO_SOT_SMD:SOT-23, F.Cu at (151.5, 52.9)
- added R23: ERJ-6GEYJ101V, Resistor_SMD:R_0805_2012Metric, F.Cu at (141.0, 48.9)
- added R24: RMCF0805JT47K0, Resistor_SMD:R_0805_2012Metric, F.Cu at (141.0, 51.9)
- added R25: RC0805FR-0751RL, Resistor_SMD:R_0805_2012Metric, F.Cu at (141.0, 54.8)
- added R6: RMCF0805JT1K80, Resistor_SMD:R_0805_2012Metric, F.Cu at (141.0, 46.0)

Commit message: #GOATED We got the KiCad symbols and footprint ;)
Parts:
- added REF**: LSM6DSOX, MM27_Custom_Footprints:LSM6DSOX, F.Cu at (44.0, 61.5)
- added REF**: LIS3MDL, MM27_Custom_Footprints:LIS3MDL, F.Cu at (59.0, 42.5)
