File: MM27/MM27.kicad_sch (KiCad schematic)
At the start: 0 parts

Commit message: power and motor control
Parts:
- added C1, C6: 10uF, Capacitor_SMD:C_0805_2012Metric_Pad1.18x1.45mm_HandSolder, symbol Device:C
- added C2: 22uF, Capacitor_SMD:C_0805_2012Metric_Pad1.18x1.45mm_HandSolder, symbol Device:C
- added C3, C5: 4.7uF, Capacitor_SMD:C_0805_2012Metric_Pad1.18x1.45mm_HandSolder, symbol Device:C
- added C4: 100nF, Capacitor_SMD:C_0805_2012Metric_Pad1.18x1.45mm_HandSolder, symbol Device:C
- added J1, J2: B2B-PH-K-S, B2B_PH_K_S:JST_B2B-PH-K-S, symbol B2B-PH-K-S:B2B-PH-K-S
- added J3, J4: Conn_01x06_Pin, Connector_JST:JST_SH_BM06B-SRSS-TB_1x06-1MP_P1.00mm_Vertical, symbol Connector:Conn_01x06_Pin
- added R1: 10k, Resistor_SMD:R_0805_2012Metric_Pad1.20x1.40mm_HandSolder, symbol Device:R
- added SW1: CL-SB-12A-01T, CL_SB_12A_01T:CL-SB-12A-01T_NDC, symbol CL_SB_12A_01T:CL-SB-12A-01T
- added U1: AZ1117IH-3.3TRG1, AZ1117IH_3_3TRG1:SOT230P700X185-4N, symbol AZ1117IH-3.3TRG1:AZ1117IH-3.3TRG1
- added U5: L293DD, L293DD:SOIC127P1032X265-20N, symbol L293DD:L293DD
Connections:
- new net: J1.2, J2.1
- new net: J1.1, SW1.3
- new net +BATT: C1.1, C3.1, C4.1, R1.1, SW1.2, U1.3 (INPUT), U5.20 (VSS)
- new net ENC1_A: J3.4 (Pin_4)
- new net ENC1_B: J3.5 (Pin_5)
- new net ENC2_A: J4.4 (Pin_4)
- new net ENC2_B: J4.5 (Pin_5)
- new net GND: C1.2, C2.2, C3.2, C4.2, C5.2, C6.2, J2.2, J3.6 (Pin_6), J4.6 (Pin_6), R1.2, SW1.1, U1.1 (GND), U5.14 (GND__4), U5.15 (GND__5), U5.16 (GND__6), U5.17 (GND__7), U5.4 (GND), U5.5 (GND__1), U5.6 (GND__2), U5.7 (GND__3)
- new net M+1: J3.1 (Pin_1), U5.3 (OUTPUT_1)
- new net M+2: J4.1 (Pin_1), U5.13 (OUTPUT_3)
- new net M-1: J3.2 (Pin_2), U5.8 (OUTPUT_2)
- new net M-2: J4.2 (Pin_2), U5.18 (OUTPUT_4)
- new net M1_C: U5.2 (INPUT_1)
- new net M1_CC: U5.9 (INPUT_2)
- new net M2_C: U5.12 (INPUT_3)
- new net M2_CC: U5.19 (INPUT_4)
- new net VCC: C2.1, C5.1, C6.1, J3.3 (Pin_3), J4.3 (Pin_3), U1.2 (OUTPUT), U1.4 (VOUT), U5.1 (ENABLE_1), U5.10 (VS), U5.11 (ENABLE_2)

Commit message: ir circuits
Parts:
- added C20: CL21B104KBCNNNC, Capacitor_SMD:C_0805_2012Metric, symbol MM_100nF:CL21B104KBCNNNC
- added C21: CL21A475KAQNNNE, Capacitor_SMD:C_0805_2012Metric, symbol MM_4.7uF:CL21A475KAQNNNE
- added LED5: INL-5AMIR15, LED_THT:LED_D3.0mm, symbol MM_IR Emitter:INL-5AMIR15
- added Q1: SFH 313 FA-3/4, LED_THT:LED_D3.0mm, symbol MM_IR Sensor:SFH_313_FA-3_4
- added Q10: NMOS, Package_TO_SOT_SMD:SOT-23, symbol Simulation_SPICE:NMOS
- added R23: ERJ-6GEYJ101V, Resistor_SMD:R_0805_2012Metric, symbol MM_100Ohm:ERJ-6GEYJ101V
- added R24: RMCF0805JT47K0, Resistor_SMD:R_0805_2012Metric, symbol MM_47kOhm:RMCF0805JT47K0
- added R25: RC0805FR-0751RL, Resistor_SMD:R_0805_2012Metric, symbol MM_51Ohm:RC0805FR-0751RL
- added R6: RMCF0805JT1K80, Resistor_SMD:R_0805_2012Metric, symbol MM_1.8kOhm:RMCF0805JT1K80
Connections:
- new net: LED5.1, Q10.1 (D)
- new net: LED5.2, R25.2
- new net: Q10.2 (G), R23.2, R24.2
- new net 3V3: C20.2, C21.2, Q1.2, R25.1
- new net AGND: R6.1
- new net GNDREF: C20.1, C21.1, Q10.3 (S), R24.1
- new net PA4: Q1.1, R6.2
- new net PC2: R23.1

Commit message: #GOATED We got the KiCad symbols and footprint ;)
Parts:
- removed U5: L293DD, L293DD:SOIC127P1032X265-20N, symbol L293DD:L293DD
- added MCU1: BlackPillv3, WeAct:WeAct-BlackPill_DIP-40_W15.24mm-SWD, symbol WeAct-BlackPillv3:WeActBlackPillV3
Connections:
- net PC2: no longer names the net of R23.1
- new net: MCU1.19 (GND), MCU1.39 (GND), MCU1.44 (GND)
- new net: MCU1.20 (3V3), MCU1.38 (3V3), MCU1.41 (3V3)
- new net 5V: MCU1.18 (5V), MCU1.40 (5V)
Other:
- moved on the sheet: C1, C2, C20, C21, J1, J2, LED5, Q1, Q10, R1, R23, R24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
